Commit message: fix(robot): align regressor body chain with caster3.xml

File: caster3/urdf/caster3.urdf (robot description, URDF)
Before this commit: robot caster3, 7 links, 6 joints
Joints:
- joint J1: limit lower=0 upper=3.14 effort=10 velocity=1 -> lower=-0.21 upper=4.47 effort=10 velocity=1
- joint J2: limit lower=0 upper=3.14 effort=10 velocity=1 -> lower=0.04 upper=3.14 effort=10 velocity=1
- joint J3: axis 0 0 1 -> 0 0 -1; limit lower=0 upper=3.14 effort=10 velocity=1 -> lower=0.04 upper=3.14 effort=10 velocity=1
- joint J4: limit lower=-2.1 upper=3.14 effort=0.8 velocity=1 -> lower=-2.2 upper=3.1 effort=0.8 velocity=1
- joint J5: limit lower=-1.57 upper=1.57 effort=0.8 velocity=1 -> lower=-1.3 upper=1.8 effort=0.8 velocity=1
- joint J6: limit lower=-1.57 upper=3.14 effort=0.8 velocity=1 -> lower=-1.9 upper=3.1 effort=0.8 velocity=1
